File: hardware/logicboard/p2-001.sch (EAGLE design)
At the start: 50 parts, among them IC1 5V, IC2 4066N, IC3 LTC485N, IC4 74LS07N, J1 LEDs, J2 Display, J3 PWR, K1 G5V1, Q1 220mA/50V/3.5Ω, Q2 220mA/50V/3.5Ω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

Commit message: DC-In connector.
Parts:
- added JV1: DC12V, SparkFun-Connectors:CONN_02-JST-2MM-SMT
Connections:
- net +12V: now also JV1.2
- net GND: now also JV1.1
Other:
- moved on the sheet: SV2-13, SV2-2, SV2-4, SV2-6, SV2-8
Changed lines of the file:
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@@
 <part name="SUPPLY39" library="supply2" deviceset="GND" device=""/>
 <part name="VDD4" library="supply1" library_urn="urn:adsk.eagle:library:371" deviceset="VDD" device=""/>
+<part name="SUPPLY40" library="supply2" deviceset="GND" device=""/>
+<part name="P+4" library="supply1" library_urn="urn:adsk.eagle:library:371" deviceset="+12V" device=""/>
+<part name="JV1" library="SparkFun-Connectors" library_urn="urn:adsk.eagle:library:513" deviceset="CONN_02" device="-JST-2MM-SMT" package3d_urn="urn:adsk.eagle:package:38042/1" value="DC12V"/>
 </parts>
 <sheets>
@@
 <attribute name="VALUE" x="342.646" y="230.759" size="1.778" layer="96"/>
 </instance>
-<instance part="SV2" gate="-2" x="342.9" y="83.82" smashed="yes">
-<attribute name="NAME" x="345.44" y="83.058" size="1.778" layer="95"/>
-<attribute name="VALUE" x="342.646" y="80.899" size="1.778" layer="96"/>
+<instance part="SV2" gate="-2" x="342.9" y="58.42" smashed="yes">
+<attribute name="NAME" x="345.44" y="57.658" size="1.778" layer="95"/>
+<attribute name="VALUE" x="342.646" y="55.499" size="1.778" layer="96"/>
 </instance>
 <instance part="SV2" gate="-3" x="342.9" y="180.34" smashed="yes">
@@
 <attribute name="VALUE" x="342.646" y="177.419" size="1.778" layer="96"/>
 </instance>
-<instance part="SV2" gate="-4" x="342.9" y="81.28" smashed="yes">
-<attribute name="NAME" x="345.44" y="80.518" size="1.778" layer="95"/>
-<attribute name="VALUE" x="342.646" y="78.359" size="1.778" layer="96"/>
+<instance part="SV2" gate="-4" x="342.9" y="55.88" smashed="yes">
+<attribute name="NAME" x="345.44" y="55.118" size="1.778" layer="95"/>
+<attribute name="VALUE" x="342.646" y="52.959" size="1.778" layer="96"/>
 </instance>
 <instance part="SV2" gate="-5" x="342.9" y="218.44" smashed="yes">
@@
 <attribute name="VALUE" x="342.646" y="215.519" size="1.778" layer="96"/>
 </instance>
-<instance part="SV2" gate="-6" x="342.9" y="78.74" smashed="yes">
-<attribute name="NAME" x="345.44" y="77.978" size="1.778" layer="95"/>
-<attribute name="VALUE" x="342.646" y="75.819" size="1.778" layer="96"/>
+<instance part="SV2" gate="-6" x="342.9" y="53.34" smashed="yes">
+<attribute name="NAME" x="345.44" y="52.578" size="1.778" layer="95"/>
+<attribute name="VALUE" x="342.646" y="50.419" size="1.778" layer="96"/>
 </instance>
 <instance part="SV2" gate="-7" x="342.9" y="203.2" smashed="yes">
@@
 <attribute name="VALUE" x="342.646" y="200.279" size="1.778" layer="96"/>
 </instance>
-<instance part="SV2" gate="-8" x="342.9" y="76.2" smashed="yes">
-<attribute name="NAME" x="345.44" y="75.438" size="1.778" layer="95"/>
-<attribute name="VALUE" x="342.646" y="73.279" size="1.778" layer="96"/>
+<instance part="SV2" gate="-8" x="342.9" y="50.8" smashed="yes">
+<attribute name="NAME" x="345.44" y="50.038" size="1.778" layer="95"/>
+<attribute name="VALUE" x="342.646" y="47.879" size="1.778" layer="96"/>
 </instance>
 <instance part="SV2" gate="-9" x="342.9" y="185.42" smashed="yes">
@@
 <attribute name="VALUE" x="342.646" y="93.599" size="1.778" layer="96"/>
 </instance>
-<instance part="SV2" gate="-13" x="342.9" y="73.66" smashed="yes">
-<attribute name="NAME" x="345.44" y="72.898" size="1.778" layer="95"/>
-<attribute name="VALUE" x="342.646" y="70.739" size="1.778" layer="96"/>
+<instance part="SV2" gate="-13" x="342.9" y="48.26" smashed="yes">
+<attribute name="NAME" x="345.44" y="47.498" size="1.778" layer="95"/>
+<attribute name="VALUE" x="342.646" y="45.339" size="1.778" layer="96"/>
 </instance>
 <instance part="SV2" gate="-14" x="342.9" y="93.98" smashed="yes">
@@
 <attribute name="VALUE" x="195.58" y="187.96" size="1.778" layer="96" align="bottom-center"/>
 </instance>
+<instance part="SUPPLY40" gate="GND" x="243.84" y="7.62" smashed="yes"/>
+<instance part="P+4" gate="1" x="243.84" y="35.56" smashed="yes">
+<attribute name="VALUE" x="238.76" y="35.56" size="1.778" layer="96" align="bottom-center"/>
+</instance>
+<instance part="JV1" gate="G$1" x="233.68" y="22.86" smashed="yes">
+<attribute name="VALUE" x="233.68" y="15.24" size="1.778" layer="96" align="bottom-center"/>
+<attribute name="NAME" x="233.68" y="30.48" size="1.778" layer="95" align="bottom-center"/>
+</instance>
 </instances>
 <busses>
@@
 <segment>
 <pinref part="SV2" gate="-2" pin="S"/>
-<wire x1="340.36" y1="83.82" x2="337.82" y2="83.82" width="0.1524" layer="91"/>
+<wire x1="340.36" y1="58.42" x2="337.82" y2="58.42" width="0.1524" layer="91"/>
 <pinref part="SUPPLY1" gate="GND" pin="GND"/>
-<wire x1="337.82" y1="83.82" x2="337.82" y2="81.28" width="0.1524" layer="91"/>
+<wire x1="337.82" y1="58.42" x2="337.82" y2="55.88" width="0.1524" layer="91"/>
 <pinref part="SV2" gate="-4" pin="S"/>
-<wire x1="337.82" y1="81.28" x2="337.82" y2="78.74" width="0.1524" layer="91"/>
-<wire x1="337.82" y1="78.74" x2="337.82" y2="76.2" width="0.1524" layer="91"/>
-<wire x1="337.82" y1="76.2" x2="337.82" y2="73.66" width="0.1524" layer="91"/>
-<wire x1="337.82" y1="73.66" x2="337.82" y2="45.72" width="0.1524" layer="91"/>
-<wire x1="340.36" y1="81.28" x2="337.82" y2="81.28" width="0.1524" layer="91"/>
-<junction x="337.82" y="81.28"/>
+<wire x1="337.82" y1="55.88" x2="337.82" y2="53.34" width="0.1524" layer="91"/>
+<wire x1="337.82" y1="53.34" x2="337.82" y2="50.8" width="0.1524" layer="91"/>
+<wire x1="337.82" y1="50.8" x2="337.82" y2="48.26" width="0.1524" layer="91"/>
+<wire x1="337.82" y1="48.26" x2="337.82" y2="45.72" width="0.1524" layer="91"/>
+<wire x1="340.36" y1="55.88" x2="337.82" y2="55.88" width="0.1524" layer="91"/>
+<junction x="337.82" y="55.88"/>
 <pinref part="SV2" gate="-6" pin="S"/>
-<wire x1="340.36" y1="78.74" x2="337.82" y2="78.74" width="0.1524" layer="91"/>
-<junction x="337.82" y="78.74"/>
+<wire x1="340.36" y1="53.34" x2="337.82" y2="53.34" width="0.1524" layer="91"/>
+<junction x="337.82" y="53.34"/>
 <pinref part="SV2" gate="-8" pin="S"/>
-<wire x1="340.36" y1="76.2" x2="337.82" y2="76.2" width="0.1524" layer="91"/>
-<junction x="337.82" y="76.2"/>
+<wire x1="340.36" y1="50.8" x2="337.82" y2="50.8" width="0.1524" layer="91"/>
+<junction x="337.82" y="50.8"/>
 <pinref part="SV2" gate="-13" pin="S"/>
-<wire x1="340.36" y1="73.66" x2="337.82" y2="73.66" width="0.1524" layer="91"/>
-<junction x="337.82" y="73.66"/>
+<wire x1="340.36" y1="48.26" x2="337.82" y2="48.26" width="0.1524" layer="91"/>
+<junction x="337.82" y="48.26"/>
 </segment>
 <segment>
@@
 <pinref part="SUPPLY39" gate="GND" pin="GND"/>
 <wire x1="198.12" y1="170.18" x2="198.12" y2="160.02" width="0.1524" layer="91"/>
+</segment>
+<segment>
+<pinref part="SUPPLY40" gate="GND" pin="GND"/>
+<wire x1="243.84" y1="22.86" x2="243.84" y2="10.16" width="0.1524" layer="91"/>
+<wire x1="241.3" y1="22.86" x2="243.84" y2="22.86" width="0.1524" layer="91"/>
+<pinref part="JV1" gate="G$1" pin="1"/>
 </segment>
 </net>
@@
 <label x="162.56" y="215.9" size="1.778" layer="95" rot="R90"/>
 </segment>
+<segment>
+<wire x1="243.84" y1="33.02" x2="243.84" y2="25.4" width="0.1524" layer="91"/>
+<pinref part="P+4" gate="1" pin="+12V"/>
+<pinref part="JV1" gate="G$1" pin="2"/>
+<wire x1="243.84" y1="25.4" x2="241.3" y2="25.4" width="0.1524" layer="91"/>
+</segment>
 </net>

Commit message: Qwiic 5V.
Parts:
- added RC5: 10k, resistor:R-EU_R2012
- added RC6: Inf, resistor:R-EU_R2012
- RC3: value 10k -> Inf
Connections:
- net SCL: now also RC4.1, RC6.1; no longer RC3.1
- net SCL3V3: now also RC5.1, RC6.2; no longer RC4.1
- net SDA: now also RC3.1
- net SDA3V3: now also RC3.2
- net VCC: now also RC4.2; no longer RC3.2
- net VDD: now also RC5.2; no longer RC4.2
Other:
- moved on the sheet: RC3, RC4
Changed lines of the file:
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@@
 <part name="VDD1" library="supply1" library_urn="urn:adsk.eagle:library:371" deviceset="VDD" device=""/>
 <part name="VDD2" library="supply1" library_urn="urn:adsk.eagle:library:371" deviceset="VDD" device=""/>
-<part name="RC3" library="resistor" library_urn="urn:adsk.eagle:library:348" deviceset="R-EU_" device="R2012" package3d_urn="urn:adsk.eagle:package:23543/2" value="10k"/>
 <part name="RC4" library="resistor" library_urn="urn:adsk.eagle:library:348" deviceset="R-EU_" device="R2012" package3d_urn="urn:adsk.eagle:package:23543/2" value="10k"/>
+<part name="RC5" library="resistor" library_urn="urn:adsk.eagle:library:348" deviceset="R-EU_" device="R2012" package3d_urn="urn:adsk.eagle:package:23543/2" value="10k"/>
 <part name="SUPPLY31" library="supply2" library_urn="urn:adsk.eagle:library:372" deviceset="VCC" device=""/>
 <part name="RC1" library="resistor" library_urn="urn:adsk.eagle:library:348" deviceset="R-EU_" device="R2012" package3d_urn="urn:adsk.eagle:package:23543/2" value="10k"/>
@@
 <part name="P+4" library="supply1" library_urn="urn:adsk.eagle:library:371" deviceset="+12V" device=""/>
 <part name="JV1" library="SparkFun-Connectors" library_urn="urn:adsk.eagle:library:513" deviceset="CONN_02" device="-JST-2MM-SMT" package3d_urn="urn:adsk.eagle:package:38042/1" value="DC12V"/>
+<part name="RC6" library="resistor" library_urn="urn:adsk.eagle:library:348" deviceset="R-EU_" device="R2012" package3d_urn="urn:adsk.eagle:package:23543/2" value="Inf"/>
+<part name="RC3" library="resistor" library_urn="urn:adsk.eagle:library:348" deviceset="R-EU_" device="R2012" package3d_urn="urn:adsk.eagle:package:23543/2" value="Inf"/>
 </parts>
 <sheets>
@@
 </instance>
 <instance part="D3" gate="G$1" x="320.04" y="160.02" smashed="yes" rot="R180">
-<attribute name="NAME" x="320.04" y="154.94" size="1.778" layer="95" font="vector" align="bottom-center"/>
+<attribute name="NAME" x="320.04" y="154.94" size="1.778" layer="95" align="bottom-center"/>
 <attribute name="VALUE" x="322.58" y="162.052" size="1.778" layer="96" font="vector" rot="R180" align="top-left"/>
 </instance>
@@
 </instance>
 <instance part="U1" gate="G$1" x="121.92" y="175.26" smashed="yes" rot="MR0">
-<attribute name="NAME" x="121.92" y="182.88" size="1.778" layer="95" font="vector" align="bottom-center"/>
-<attribute name="VALUE" x="121.92" y="165.1" size="1.778" layer="96" font="vector" rot="MR0" align="bottom-center"/>
+<attribute name="NAME" x="121.92" y="182.88" size="1.778" layer="95" align="bottom-center"/>
+<attribute name="VALUE" x="121.92" y="165.1" size="1.778" layer="96" rot="MR0" align="bottom-center"/>
 </instance>
 <instance part="K1" gate="1" x="119.38" y="228.6" smashed="yes">
@@
 </instance>
 <instance part="D1" gate="G$1" x="127" y="228.6" smashed="yes" rot="R90">
-<attribute name="NAME" x="132.08" y="228.6" size="1.778" layer="95" font="vector" align="bottom-center"/>
+<attribute name="NAME" x="132.08" y="228.6" size="1.778" layer="95" align="bottom-center"/>
 <attribute name="VALUE" x="129.032" y="226.06" size="1.778" layer="96" font="vector" rot="R90" align="top-left"/>
 </instance>
@@
 </instance>
 <instance part="Q2" gate="NMOS" x="180.34" y="134.62" smashed="yes" rot="MR270">
-<attribute name="NAME" x="180.34" y="129.54" size="1.778" layer="95" font="vector" rot="MR0" align="bottom-center"/>
-<attribute name="VALUE" x="180.34" y="127" size="1.778" layer="96" font="vector" rot="MR0" align="bottom-center"/>
+<attribute name="NAME" x="180.34" y="139.7" size="1.778" layer="95" rot="MR0" align="bottom-center"/>
+<attribute name="VALUE" x="180.34" y="144.78" size="1.778" layer="96" rot="MR0" align="bottom-center"/>
 </instance>
 <instance part="VDD1" gate="G$1" x="170.18" y="243.84" smashed="yes">
@@
 <attribute name="VALUE" x="182.88" y="154.94" size="1.778" layer="96" align="bottom-center"/>
 </instance>
-<instance part="RC3" gate="G$1" x="172.72" y="139.7" smashed="yes" rot="R90">
+<instance part="RC4" gate="G$1" x="172.72" y="139.7" smashed="yes" rot="R90">
 <attribute name="NAME" x="170.18" y="139.7" size="1.778" layer="95" rot="R90" align="bottom-center"/>
 <attribute name="VALUE" x="175.26" y="139.7" size="1.778" layer="96" rot="R90" align="bottom-center"/>
 </instance>
-<instance part="RC4" gate="G$1" x="187.96" y="139.7" smashed="yes" rot="R90">
+<instance part="RC5" gate="G$1" x="187.96" y="139.7" smashed="yes" rot="R90">
 <attribute name="NAME" x="185.42" y="139.7" size="1.778" layer="95" rot="R90" align="bottom-center"/>
 <attribute name="VALUE" x="190.5" y="139.7" size="1.778" layer="96" rot="R90" align="bottom-center"/>
@@
 </instance>
 <instance part="Q1" gate="NMOS" x="180.34" y="167.64" smashed="yes" rot="MR270">
-<attribute name="NAME" x="180.34" y="162.56" size="1.778" layer="95" font="vector" rot="MR0" align="bottom-center"/>
-<attribute name="VALUE" x="180.34" y="160.02" size="1.778" layer="96" font="vector" rot="MR0" align="bottom-center"/>
+<attribute name="NAME" x="180.34" y="172.72" size="1.778" layer="95" rot="MR0" align="bottom-center"/>
+<attribute name="VALUE" x="180.34" y="177.8" size="1.778" layer="96" rot="MR0" align="bottom-center"/>
 </instance>
 <instance part="VDD3" gate="G$1" x="182.88" y="185.42" smashed="yes">
@@
 </instance>
 <instance part="JQ1" gate="J1" x="208.28" y="167.64" smashed="yes" rot="R180">
-<attribute name="VALUE" x="208.28" y="157.48" size="1.778" layer="96" font="vector" align="bottom-center"/>
-<attribute name="NAME" x="208.28" y="175.006" size="1.778" layer="95" font="vector" align="bottom-center"/>
+<attribute name="VALUE" x="208.28" y="157.48" size="1.778" layer="96" align="bottom-center"/>
+<attribute name="NAME" x="208.28" y="175.006" size="1.778" layer="95" align="bottom-center"/>
 </instance>
 <instance part="SUPPLY39" gate="GND" x="198.12" y="157.48" smashed="yes"/>
@@
 <attribute name="VALUE" x="233.68" y="15.24" size="1.778" layer="96" align="bottom-center"/>
 <attribute name="NAME" x="233.68" y="30.48" size="1.778" layer="95" align="bottom-center"/>
+</instance>
+<instance part="RC6" gate="G$1" x="180.34" y="127" smashed="yes">
+<attribute name="NAME" x="180.34" y="129.54" size="1.778" layer="95" align="bottom-center"/>
+<attribute name="VALUE" x="180.34" y="124.46" size="1.778" layer="96" align="bottom-center"/>
+</instance>
+<instance part="RC3" gate="G$1" x="180.34" y="160.02" smashed="yes">
+<attribute name="NAME" x="180.34" y="162.56" size="1.778" layer="95" align="bottom-center"/>
+<attribute name="VALUE" x="180.34" y="157.48" size="1.778" layer="96" align="bottom-center"/>
 </instance>
 </instances>
@@
 </segment>
 <segment>
-<pinref part="RC3" gate="G$1" pin="2"/>
+<pinref part="RC4" gate="G$1" pin="2"/>
 <pinref part="SUPPLY31" gate="G$1" pin="VCC"/>
 <wire x1="172.72" y1="147.32" x2="172.72" y2="144.78" width="0.1524" layer="91"/>
@@
 <junction x="172.72" y="165.1"/>
 <label x="157.48" y="165.1" size="1.778" layer="95"/>
+<pinref part="RC3" gate="G$1" pin="1"/>
+<wire x1="175.26" y1="160.02" x2="172.72" y2="160.02" width="0.1524" layer="91"/>
+<wire x1="172.72" y1="160.02" x2="172.72" y2="165.1" width="0.1524" layer="91"/>
 </segment>
 </net>
@@
 <wire x1="157.48" y1="132.08" x2="172.72" y2="132.08" width="0.1524" layer="91"/>
 <label x="157.48" y="132.08" size="1.778" layer="95"/>
-<pinref part="RC3" gate="G$1" pin="1"/>
+<pinref part="RC4" gate="G$1" pin="1"/>
 <wire x1="172.72" y1="132.08" x2="175.26" y2="132.08" width="0.1524" layer="91"/>
 <wire x1="172.72" y1="134.62" x2="172.72" y2="132.08" width="0.1524" layer="91"/>
 <junction x="172.72" y="132.08"/>
+<pinref part="RC6" gate="G$1" pin="1"/>
+<wire x1="175.26" y1="127" x2="172.72" y2="127" width="0.1524" layer="91"/>
+<wire x1="172.72" y1="127" x2="172.72" y2="132.08" width="0.1524" layer="91"/>
 </segment>
 </net>
@@
 <pinref part="VDD2" gate="G$1" pin="VDD"/>
 <wire x1="182.88" y1="149.86" x2="182.88" y2="147.32" width="0.1524" layer="91"/>
-<pinref part="RC4" gate="G$1" pin="2"/>
+<pinref part="RC5" gate="G$1" pin="2"/>
 <wire x1="182.88" y1="147.32" x2="182.88" y2="139.7" width="0.1524" layer="91"/>
 <wire x1="187.96" y1="144.78" x2="187.96" y2="147.32" width="0.1524" layer="91"/>
@@
 <pinref part="Q2" gate="NMOS" pin="S"/>
 <wire x1="185.42" y1="132.08" x2="187.96" y2="132.08" width="0.1524" layer="91"/>
-<pinref part="RC4" gate="G$1" pin="1"/>
+<pinref part="RC5" gate="G$1" pin="1"/>
 <wire x1="187.96" y1="132.08" x2="193.04" y2="132.08" width="0.1524" layer="91"/>
 <wire x1="187.96" y1="134.62" x2="187.96" y2="132.08" width="0.1524" layer="91"/>
@@
 <wire x1="200.66" y1="162.56" x2="193.04" y2="162.56" width="0.1524" layer="91"/>
 <wire x1="193.04" y1="162.56" x2="193.04" y2="132.08" width="0.1524" layer="91"/>
+<pinref part="RC6" gate="G$1" pin="2"/>
+<wire x1="185.42" y1="127" x2="187.96" y2="127" width="0.1524" layer="91"/>
+<wire x1="187.96" y1="127" x2="187.96" y2="132.08" width="0.1524" layer="91"/>
 </segment>
 </net>
@@
 <wire x1="200.66" y1="165.1" x2="187.96" y2="165.1" width="0.1524" layer="91"/>
 <junction x="187.96" y="165.1"/>
-</segment>
-</net>
+<pinref part="RC3" gate="G$1" pin="2"/>
+<wire x1="185.42" y1="160.02" x2="187.96" y2="160.02" width="0.1524" layer="91"/>
+<wire x1="187.96" y1="160.02" x2="187.96" y2="165.1" width="0.1524" layer="91"/>
+</segment>
+</net>
