File: hardware/logicboard/p2-001.brd (EAGLE design)
At the start: 72 x 72 mm, 58 parts, among them IC1 74LS07N, IC11 74LS153D, IC12 LTC485S, IC13 LTC485S, IC2 4066N, J1 DISP, J11 Qwiic, J12 Qwiic, J13 Qwiic, J14 Qwiic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

Commit message: Looks good.
Parts:
- removed JP5: GNDPIN, pinhead:1X01
- removed R4: 1k, resistor:0204/5
- added JP2: MPXJMP, pinhead:1X02
- JP4: value MPXJMP -> GNDPIN; device pinhead:1X02 -> pinhead:1X01
- moved JP4 11.2 mm to (65.0, 69.0), turned to 0 degrees
Connections:
- removed net PWRLED: R4.1, SV2.5
- net +9V: no longer R4.2
- net D7: now also J2.4; no longer J2.2
- net DISP1: now also J1.2; no longer J1.1
- net DISP2: now also J1.3; no longer J1.2
- net GND: now also J1.1, J2.1, JP4.1; no longer J1.3, J2.5, JP5.1
- net MIN: now also JP2.2; no longer JP4.2
- net RX: now also JP2.1; no longer JP4.1
- net SDA: now also J2.2; no longer J2.4
- net VCC: now also J2.5; no longer J2.1
Routing:
- net PWRLED: track 71.5 -> 0.00 mm
- net LED1: track 53.1 -> 106.6 mm, vias 1 -> 0
- net MIN: track 84.9 -> 124.0 mm, vias 5 -> 2
- net MTX-: track 108.0 -> 69.0 mm, vias 0 -> 2
- net SCL: track 175.3 -> 207.0 mm, vias 7 -> 6
- net +9VB: track 58.9 -> 87.2 mm
- net +9V: track 137.8 -> 116.0 mm, vias 4 -> 1
- net VDD: track 64.8 -> 84.1 mm, vias 0 -> 2
- net MRX-: track 52.0 -> 70.5 mm
- net DISP1: track 54.9 -> 38.9 mm, vias 1 -> 0
- net GND: track 434.5 -> 418.8 mm, vias 5 -> 3
- net DTCT1: track 37.5 -> 52.8 mm
- net +5V: track 86.4 -> 100.1 mm, vias 1 -> 2
- net THS: track 70.8 -> 58.1 mm, vias 2 -> 1
- net LED0: track 71.1 -> 59.4 mm, vias 1 -> 3
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Other:
- board text added: "JP1"
- board text added: "JP2"
- board text added: "Remove JP2"
- board text removed: "JP4"
- board text removed: "Remove JP4"

Commit message: Removed bus.
Parts:
- J1: value DISP -> GPIO
- J2: value I2C -> MKR
Connections:
- net DISP1 renamed GPIO1
- net DISP2 renamed GPIO2
- net LED1A renamed N$6
- net MINRTN renamed MIRETN
- net MINSND renamed MISEND
- removed net +3V3: J4.3, MC1.P$33
- removed net +5V: F1.1, R3.2, SV1.1, SV1.13, SV1.5, SV1.9
- removed net +9V: JP1.1, K1.1, SV2.1
- removed net +9VB: C3.1, C4.1, D1.C, JP1.2, K1.5, K1.6, V1.IN
- removed net ANLG1PDN: IC2.2, RN3.2
- removed net ANLG2PDN: IC2.3, RN3.3
- removed net ANLG3PDN: IC2.9, RN3.4
- removed net LED0A: J3.1, R5.1
- removed net MISO: MC1.P$19
- removed net MOSI: MC1.P$17
- removed net SCLK: MC1.P$18
- removed net SS: MC1.P$16
- new net N$1: IC2.10, RN3.2
- new net N$3: IC2.3, RN3.4
- new net N$4: F1.1, JP1.1, K1.1
- new net N$5: IC2.2, RN3.5
- new net N$7: J3.3, R5.1
- new net V5V: F1.2, R3.2, SV1.1, SV1.13, SV1.5, SV1.9
- new net VIN: C3.1, C4.1, D1.C, J4.1, SV2.1, V1.IN
- net GND: now also J3.1; no longer J3.3
- net LED0: now also R6.2; no longer R5.2
- net LED1: now also R5.2; no longer R6.2
- net N$2: now also IC2.9, RN3.3; no longer IC2.10, RN3.5
- net VCC: now also JP1.2, K1.5, K1.6; no longer F1.2
- net VDD: now also J4.3, MC1.P$33; no longer J4.1, MC1.P$20
Routing:
- net VIN: track 0.00 -> 146.5 mm, vias 0 -> 1
- net +9V: track 116.0 -> 0.00 mm, vias 1 -> 0
- net +5V: track 100.1 -> 0.00 mm, vias 2 -> 0
- net +9VB: track 87.2 -> 0.00 mm, vias 1 -> 0
- net V5V: track 0.00 -> 79.6 mm, vias 0 -> 2
- net VDD: track 84.1 -> 30.2 mm
- net MRX-: track 70.5 -> 35.9 mm, vias 0 -> 2
- net SCL: track 207.0 -> 172.7 mm, vias 6 -> 2
- net MIN: track 124.0 -> 89.8 mm
- net GND: track 418.8 -> 451.1 mm, vias 3 -> 2
- net N$5: track 0.00 -> 30.5 mm
- net +3V3: track 28.9 -> 0.00 mm
- net VCC: track 380.0 -> 353.8 mm, vias 8 -> 6
- net ANLG1PDN: track 24.5 -> 0.00 mm
- net MIRETN: track 67.3 -> 45.8 mm, vias 0 -> 1
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
Commit message: A little bit better.
Connections:
- new net N$10: J13.1
- net GND: no longer J13.1
Routing:
- net GND: track 451.1 -> 436.2 mm

Commit message: Rough design. Looks okay.
Parts:
- J1: value GPIO -> MKR; device SparkFun-Connectors:JST-3-PTH-VERT -> SparkFun-Connectors:JST-5-PTH
- J2: value MKR -> GPIO; device SparkFun-Connectors:JST-5-PTH -> SparkFun-Connectors:JST-3-PTH-VERT
- JP1: value RLYJMP -> RTC; device pinhead:1X02 -> SparkFun-Connectors:1X05
- JP3: value RTC -> RLYJMP; device SparkFun-Connectors:1X05 -> pinhead:1X02
- moved JP1 40.9 mm to (23.8, 53.3)
- moved JP3 40.9 mm to (17.0, 13.0)
- moved C11 33.0 mm to (36.0, 7.00)
- moved C13 33.0 mm to (36.0, 40.0)
- moved R12 19.3 mm to (32.5, 31.0)
- moved R13 19.3 mm to (36.0, 50.0)
- moved IC12 19.0 mm to (36.0, 26.0)
- moved IC13 19.0 mm to (36.0, 45.0)
- moved J1 17.2 mm to (66.0, 59.0), turned to 270 degrees
- moved J2 17.2 mm to (52.0, 69.0), turned to 0 degrees
Connections:
- net MO1RTN renamed MO1RETN
- net MO1SND renamed MO1SEND
- net MO2RTN renamed MO2RETN
- net MO2SND renamed MO2SEND
- net MTHRTN renamed MTRETN
- net MTHSND renamed MTSEND
- net D7: now also J1.4; no longer J2.4
- net GND: now also IC12.2, IC12.3, IC12.4, JP1.2; no longer IC13.2, IC13.3, IC13.4, JP3.2
- net GPIO1: now also J2.2; no longer J1.2
- net GPIO2: now also J2.3; no longer J1.3
- net MRX: now also IC12.1; no longer IC13.1
- net MRX+: now also IC12.6, R12.1; no longer IC13.6, R13.1
- net MRX-: now also IC12.7, R12.2; no longer IC13.7, R13.2
- net MTX+: now also IC13.6, R13.1; no longer IC12.6, R12.1
- net MTX-: now also IC13.7, R13.2; no longer IC12.7, R12.2
- net N$4: now also JP3.1; no longer JP1.1
- net SCL: now also J1.3, JP1.4; no longer J2.3, JP3.4
- net SDA: now also J1.2, JP1.5; no longer J2.2, JP3.5
- net TX: now also IC13.4; no longer IC12.4
- net VCC: now also IC13.2, IC13.3, J1.5, JP1.1, JP3.2; no longer IC12.2, IC12.3, J2.5, JP1.2, JP3.1
Routing:
- net GND: track 436.2 -> 0.00 mm, vias 2 -> 0
- net VCC: track 353.8 -> 0.00 mm, vias 6 -> 0
- net SDA: track 206.4 -> 0.00 mm, vias 5 -> 0
- net SCL: track 172.7 -> 0.00 mm, vias 2 -> 0
- net VIN: track 146.5 -> 0.00 mm, vias 1 -> 0
- net RX: track 107.8 -> 0.00 mm, vias 3 -> 0
- net MTX+: track 103.2 -> 0.00 mm, vias 2 -> 0
- net LED1: track 92.6 -> 0.00 mm, vias 1 -> 0
- net MIN: track 89.8 -> 0.00 mm, vias 2 -> 0
- net V5V: track 79.6 -> 0.00 mm, vias 2 -> 0
- net LED0: track 73.2 -> 0.00 mm
- net THS: track 59.3 -> 0.00 mm, vias 2 -> 0
- net TX: track 57.8 -> 0.00 mm, vias 1 -> 0
- net MTX-: track 57.0 -> 0.00 mm, vias 2 -> 0
- net ANLG1: track 52.2 -> 0.00 mm
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- removed copper zone on layer 1, net GND
- removed copper zone on layer 16, net GND
Other:
- board text added: "GPIO1"
- board text added: "GPIO2"
- board text removed: "DISP1"
- board text removed: "DISP2"

Commit message: Refine.
Parts:
- turned C9 to 180 degrees
Connections:
- net MTH renamed MT
- net N$4 renamed V5VRAW
- removed net N$10: J13.1
- net GND: now also J13.1
Routing:
- net GND: track 0.00 -> 439.6 mm, vias 0 -> 1
- net VCC: track 0.00 -> 380.0 mm, vias 0 -> 5
- net SCL: track 0.00 -> 191.8 mm, vias 0 -> 1
- net SDA: track 0.00 -> 186.4 mm, vias 0 -> 6
- net VIN: track 0.00 -> 149.2 mm, vias 0 -> 2
- net RX: track 0.00 -> 113.9 mm, vias 0 -> 2
- net MTX-: track 0.00 -> 111.1 mm
- net MTX+: track 0.00 -> 101.4 mm, vias 0 -> 2
- net V5V: track 0.00 -> 94.5 mm
- net MIN: track 0.00 -> 89.8 mm, vias 0 -> 3
- net LED0: track 0.00 -> 72.5 mm
- net MRXDTCT: track 0.00 -> 67.4 mm, vias 0 -> 3
- net TX: track 0.00 -> 67.1 mm, vias 0 -> 1
- net GPIO1: track 0.00 -> 61.0 mm
- net MIRETN: track 0.00 -> 61.0 mm
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- added copper zone on layer 1, net GND
- added copper zone on layer 16, net GND

Commit message: Changed power supply.
Connections:
- new net VOUT: C1.1, C2.1, D1.A, JP3.2, K1.5, K1.6, V1.OUT
- net VCC: no longer C1.1, C2.1, D1.A, JP3.2, K1.5, K1.6, V1.OUT
- net VIN: now also MC1.P$20
Routing:
- net VOUT: track 0.00 -> 70.6 mm
- net MTX-: track 111.1 -> 56.4 mm, vias 0 -> 2
- net MTX+: track 101.4 -> 59.3 mm, vias 2 -> 4
- net VCC: track 380.0 -> 339.8 mm, vias 5 -> 7
- net LED1: track 58.1 -> 89.2 mm, vias 4 -> 3
- net SDA: track 186.4 -> 156.4 mm, vias 6 -> 11
- net THS: track 60.5 -> 85.5 mm, vias 1 -> 2
- net VIN: track 149.2 -> 172.9 mm, vias 2 -> 0
- net GPIO1: track 61.0 -> 40.9 mm, vias 0 -> 1
- net RX: track 113.9 -> 132.6 mm, vias 2 -> 1
- net GND: track 439.6 -> 457.3 mm, vias 1 -> 3
- net N$5: track 20.8 -> 30.5 mm, vias 1 -> 0
- net V5V: track 94.5 -> 103.0 mm
- net ANLG1: track 38.2 -> 45.7 mm, vias 1 -> 0
- net MIN: track 89.8 -> 95.5 mm, vias 3 -> 2
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
Commit message: Added power selector.
Parts:
- added JP5: GNDPIN, pinhead:1X01
- C1: value 1u -> 22u; device rcl:C050-024X044 -> rcl:C025-050X050
- C2: value 100n -> 470n; device rcl:C025-024X044 -> rcl:C050-024X044
- C3: value 470n -> 1u
- C4: value 22u -> 100n; device rcl:C025-050X050 -> rcl:C025-024X044
- JP4: value GNDPIN -> PWRSEL; device pinhead:1X01 -> pinhead:1X03
- moved JP4 51.4 mm to (15.0, 57.0)
- moved C4 21.9 mm to (52.0, 19.0), turned to 180 degrees
- moved C1 12.1 mm to (36.0, 4.00), turned to 0 degrees
- moved C3 8.00 mm to (47.0, 9.00)
- moved C2 5.39 mm to (47.0, 17.0), turned to 270 degrees
Connections:
- net V5VRAW renamed N$4
- new net VOUTRAW: C3.1, C4.1, D1.A, JP3.2, K1.5, K1.6, V1.OUT
- net GND: now also JP5.1; no longer JP4.1
- net V5V: now also JP4.2; no longer F1.2
- net VCC: now also JP4.3
- net VIN: now also C1.1, C2.1; no longer C3.1, C4.1
- net VOUT: now also F1.2, JP4.1; no longer C1.1, C2.1, D1.A, JP3.2, K1.5, K1.6, V1.OUT
Routing:
- net VOUTRAW: track 0.00 -> 60.0 mm
- net MTX-: track 56.4 -> 110.3 mm, vias 2 -> 0
- net V5V: track 103.0 -> 55.8 mm, vias 0 -> 1
- net VCC: track 339.8 -> 371.7 mm, vias 7 -> 8
- net MTX+: track 59.3 -> 91.1 mm, vias 4 -> 2
- net LED0: track 67.6 -> 96.2 mm
- net MRXDTCT: track 66.6 -> 47.5 mm, vias 2 -> 5
- net THS: track 85.5 -> 68.2 mm, vias 2 -> 1
- net RX: track 132.6 -> 116.8 mm, vias 1 -> 2
- net SCL: track 188.9 -> 173.7 mm, vias 5 -> 3
- net TX: track 66.5 -> 79.3 mm
- net GND: track 457.3 -> 446.2 mm, vias 3 -> 2
- net MRX+: track 36.1 -> 46.6 mm
- net VIN: track 172.9 -> 163.8 mm, vias 0 -> 2
- net MIN: track 95.5 -> 99.5 mm, vias 2 -> 1
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Other:
- board text added: "ARD"
- board text added: "JP4"
- board text added: "REG"

Commit message: Added relay-out connector (again).
Parts:
- added J5: RLY, SparkFun-Connectors:JST-2-PTH
- moved J4 35.5 mm to (36.0, 69.5), turned to 0 degrees
- moved J2 0.50 mm to (52.0, 69.5)
Connections:
- new net RLYOUT: J5.1, K1.10
- net VOUTRAW: now also J5.2
Routing:
- net MTX-: track 110.3 -> 58.1 mm, vias 0 -> 4
- net VOUTRAW: track 60.0 -> 111.7 mm, vias 0 -> 3
- net RLYOUT: track 0.00 -> 45.0 mm, vias 0 -> 2
- net TX: track 79.3 -> 52.9 mm
- net LED1: track 90.3 -> 69.8 mm, vias 2 -> 0
- net SDA: track 154.4 -> 172.2 mm
- net VOUT: track 72.2 -> 89.1 mm, vias 0 -> 1
- net LED0: track 96.2 -> 79.6 mm, vias 1 -> 2
- net GND: track 446.2 -> 433.5 mm, vias 2 -> 5
- net RX: track 116.8 -> 104.7 mm, vias 2 -> 5
- net MRX+: track 46.6 -> 36.0 mm, vias 0 -> 1
- net MTX+: track 91.1 -> 101.1 mm
- net V5V: track 55.8 -> 65.3 mm, vias 1 -> 0
- net DTCT3: track 50.5 -> 41.0 mm, vias 0 -> 1
- net VCC: track 371.7 -> 362.3 mm, vias 8 -> 9
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Other:
- board text added: "2.0.3-B"
- board text added: "3V"
- board text added: "9V"
- board text added: "G1"
- board text added: "G2"
- board text added: "RLY1"
- board text added: "RLY2"
- board text removed: "2.0.3-A"
- board text removed: "3.3V"
- board text removed: "GPIO1"
- board text removed: "GPIO2"
- board text removed: "Vin"
