File: hardware/logicboard/p2-003.brd (EAGLE design)
At the start: 91 x 90 mm, 52 parts, among them IC1 74LS06N, IC2 4066N, J1 MKR, J2 GPIO, J3 Vcc, J4 RLY, J5 SPI, J7 DIN5, J8 DIN5, J9 DIN5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

Commit message: Renumbered some connectors.
Parts:
- removed X3: MKDSN1,5/2-5,08, con-phoenix-508:MKDSN1,5/2-5,08
- JP5: device pinhead:1X02 -> pinhead:1X03
- moved JP5 82.1 mm to (87.0, 20.5), turned to 90 degrees
- moved JP3 63.2 mm to (76.0, 34.0), turned to 90 degrees
- renumbered J10 to J0
Connections:
- net GND: now also JP5.1; no longer X3.1
- net V+: now also JP5.3; no longer X3.2
- net VCC: now also JP5.2
Routing:
- net GND: track 324.0 -> 0.00 mm, vias 2 -> 0
- net VCC: track 265.4 -> 0.00 mm, vias 3 -> 0
- net VCC/2: track 132.8 -> 0.00 mm
- net V+: track 118.1 -> 0.00 mm
- net AREF: track 111.4 -> 0.00 mm, vias 2 -> 0
- net SDA: track 108.2 -> 0.00 mm, vias 3 -> 0
- net SCL: track 97.6 -> 0.00 mm, vias 4 -> 0
- net THS: track 96.9 -> 0.00 mm, vias 1 -> 0
- net ANLG3: track 93.7 -> 0.00 mm
- net LED0: track 93.4 -> 0.00 mm, vias 3 -> 0
- net GPIO1: track 79.0 -> 0.00 mm, vias 1 -> 0
- net GPIO2: track 77.2 -> 0.00 mm, vias 1 -> 0
- net RST: track 72.4 -> 0.00 mm
- net LED1: track 69.7 -> 0.00 mm, vias 1 -> 0
- net ANLG4: track 65.9 -> 0.00 mm
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Other:
- board text added: "RST"
- board text removed: "RTC1"
