File: peripheral/port-replicator/hardware/logicboard/p20-001.sch (EAGLE design)
At the start: 21 parts, among them IC1 74LS07N, J1 AUDIO_JACK_3.5MM_PTH, J11 DIN5, J12 DIN5, J13 DIN5, J2 AUDIO_JACK_3.5MM_PTH, J3 AUDIO_JACK_3.5MM_PTH, J4 AUDIO_JACK_3.5MM_PTH

Commit message: Port replicator.
Parts:
- J0: value (none) -> DC9V
- LED1: value (none) -> PWR
- LED2: value (none) -> IN
- LED3: value (none) -> OUT
Connections:
- removed net ANGL4R: J4.RING
- net ANLG4R: now also J4.RING
- net GND: now also IC1P.GND
- net VCC: now also IC1P.VCC
Changed lines of the file:
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@@
 <part name="J12" library="SparkFun-Connectors" library_urn="urn:adsk.eagle:library:513" deviceset="DIN5" device="" package3d_urn="urn:adsk.eagle:package:38294/1"/>
 <part name="J13" library="SparkFun-Connectors" library_urn="urn:adsk.eagle:library:513" deviceset="DIN5" device="" package3d_urn="urn:adsk.eagle:package:38294/1"/>
-<part name="J0" library="con-jack" library_urn="urn:adsk.eagle:library:154" deviceset="JACK-PLUG" device="0" package3d_urn="urn:adsk.eagle:package:7492/1"/>
+<part name="J0" library="con-jack" library_urn="urn:adsk.eagle:library:154" deviceset="JACK-PLUG" device="0" package3d_urn="urn:adsk.eagle:package:7492/1" value="DC9V"/>
 <part name="J1" library="SparkFun-Connectors" library_urn="urn:adsk.eagle:library:513" deviceset="AUDIO_JACK_3.5MM" device="_PTH" package3d_urn="urn:adsk.eagle:package:37997/1"/>
 <part name="J2" library="SparkFun-Connectors" library_urn="urn:adsk.eagle:library:513" deviceset="AUDIO_JACK_3.5MM" device="_PTH" package3d_urn="urn:adsk.eagle:package:37997/1"/>
@@
 <part name="R1" library="rcl" library_urn="urn:adsk.eagle:library:334" deviceset="R-EU_" device="0204/5" package3d_urn="urn:adsk.eagle:package:23488/1"/>
 <part name="R2" library="rcl" library_urn="urn:adsk.eagle:library:334" deviceset="R-EU_" device="0204/5" package3d_urn="urn:adsk.eagle:package:23488/1"/>
-<part name="LED1" library="led" library_urn="urn:adsk.eagle:library:259" deviceset="LED" device="3MM" package3d_urn="urn:adsk.eagle:package:15797/1"/>
-<part name="LED2" library="led" library_urn="urn:adsk.eagle:library:259" deviceset="LED" device="3MM" package3d_urn="urn:adsk.eagle:package:15797/1"/>
-<part name="LED3" library="led" library_urn="urn:adsk.eagle:library:259" deviceset="LED" device="3MM" package3d_urn="urn:adsk.eagle:package:15797/1"/>
+<part name="LED1" library="led" library_urn="urn:adsk.eagle:library:259" deviceset="LED" device="3MM" package3d_urn="urn:adsk.eagle:package:15797/1" value="PWR"/>
+<part name="LED2" library="led" library_urn="urn:adsk.eagle:library:259" deviceset="LED" device="3MM" package3d_urn="urn:adsk.eagle:package:15797/1" value="IN"/>
+<part name="LED3" library="led" library_urn="urn:adsk.eagle:library:259" deviceset="LED" device="3MM" package3d_urn="urn:adsk.eagle:package:15797/1" value="OUT"/>
 <part name="R3" library="rcl" library_urn="urn:adsk.eagle:library:334" deviceset="R-EU_" device="0204/5" package3d_urn="urn:adsk.eagle:package:23488/1"/>
+<part name="SUPPLY1" library="supply2" deviceset="GND" device=""/>
 </parts>
 <sheets>
@@
 <attribute name="VALUE" x="255.27" y="136.398" size="1.778" layer="96"/>
 </instance>
+<instance part="IC1" gate="P" x="241.3" y="213.36" smashed="yes">
+<attribute name="NAME" x="240.665" y="212.725" size="1.778" layer="95"/>
+</instance>
+<instance part="SUPPLY1" gate="GND" x="241.3" y="195.58" smashed="yes"/>
 </instances>
 <busses>
@@
 <label x="43.18" y="157.48" size="0.8128" layer="95" rot="R270" xref="yes"/>
 </segment>
+<segment>
+<pinref part="IC1" gate="P" pin="GND"/>
+<wire x1="241.3" y1="203.2" x2="241.3" y2="198.12" width="0.1524" layer="91"/>
+<pinref part="SUPPLY1" gate="GND" pin="GND"/>
+</segment>
 </net>
 <net name="VCC" class="2">
@@
 <label x="279.4" y="157.48" size="0.8128" layer="95" xref="yes"/>
 </segment>
+<segment>
+<pinref part="IC1" gate="P" pin="VCC"/>
+<wire x1="241.3" y1="223.52" x2="241.3" y2="226.06" width="0.1524" layer="91"/>
+<label x="241.3" y="226.06" size="0.8128" layer="95" rot="R90" xref="yes"/>
+</segment>
 </net>
 <net name="MTX+" class="0">
@@
 <label x="43.18" y="78.74" size="0.8128" layer="95" xref="yes"/>
 </segment>
+<segment>
+<pinref part="J4" gate="G$1" pin="RING"/>
+<wire x1="96.52" y1="55.88" x2="99.06" y2="55.88" width="0.1524" layer="91"/>
+<label x="99.06" y="55.88" size="0.8128" layer="95" xref="yes"/>
+</segment>
 </net>
 <net name="MTSND" class="0">
@@
 </segment>
 </net>
-<net name="ANGL4R" class="0">
-<segment>
-<pinref part="J4" gate="G$1" pin="RING"/>
-<wire x1="96.52" y1="55.88" x2="99.06" y2="55.88" width="0.1524" layer="91"/>
-<label x="99.06" y="55.88" size="0.8128" layer="95" xref="yes"/>
-</segment>
-</net>

Commit message: The port replicator now has euroblock terminal.
Parts:
- added X0: MKDSN1,5/2-5,08, con-phoenix-508:MKDSN1,5/2-5,08
Connections:
- net DTCT1: now also JP1.2; no longer JP1.1
- net DTCT2: now also JP1.4; no longer JP1.3
- net DTCT3: now also JP1.6; no longer JP1.5
- net DTCT4: now also JP1.8; no longer JP1.7
- net GND: now also JP1.1, JP1.3, JP1.5, JP1.7, X0-1.KL; no longer JP1.2, JP1.4, JP1.6, JP1.8
- net V+: now also X0-2.KL
Changed lines of the file:
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@@
 <part name="R3" library="rcl" library_urn="urn:adsk.eagle:library:334" deviceset="R-EU_" device="0204/5" package3d_urn="urn:adsk.eagle:package:23488/1"/>
 <part name="SUPPLY1" library="supply2" deviceset="GND" device=""/>
+<part name="X0" library="con-phoenix-508" library_urn="urn:adsk.eagle:library:176" deviceset="MKDSN1,5/2-5,08" device="" package3d_urn="urn:adsk.eagle:package:9630/1"/>
 </parts>
 <sheets>
@@
 </instance>
 <instance part="SUPPLY1" gate="GND" x="241.3" y="195.58" smashed="yes"/>
+<instance part="X0" gate="-1" x="38.1" y="223.52" smashed="yes" rot="MR0">
+<attribute name="NAME" x="35.052" y="222.631" size="1.778" layer="95" rot="MR0"/>
+<attribute name="VALUE" x="40.64" y="219.837" size="1.778" layer="96" rot="MR0"/>
+</instance>
+<instance part="X0" gate="-2" x="38.1" y="218.44" smashed="yes" rot="MR0">
+<attribute name="NAME" x="35.052" y="217.551" size="1.778" layer="95" rot="MR0"/>
+<attribute name="VALUE" x="40.64" y="214.757" size="1.778" layer="96" rot="MR0"/>
+</instance>
 </instances>
 <busses>
@@
 <wire x1="96.52" y1="58.42" x2="99.06" y2="58.42" width="0.1524" layer="91"/>
 <label x="99.06" y="58.42" size="0.8128" layer="95" xref="yes"/>
-</segment>
-<segment>
-<pinref part="JP1" gate="A" pin="2"/>
-<wire x1="99.06" y1="25.4" x2="104.14" y2="25.4" width="0.1524" layer="91"/>
-<pinref part="JP1" gate="A" pin="4"/>
-<wire x1="99.06" y1="22.86" x2="104.14" y2="22.86" width="0.1524" layer="91"/>
-<wire x1="104.14" y1="22.86" x2="104.14" y2="25.4" width="0.1524" layer="91"/>
-<pinref part="JP1" gate="A" pin="6"/>
-<wire x1="99.06" y1="20.32" x2="104.14" y2="20.32" width="0.1524" layer="91"/>
-<wire x1="104.14" y1="20.32" x2="104.14" y2="22.86" width="0.1524" layer="91"/>
-<junction x="104.14" y="22.86"/>
-<pinref part="JP1" gate="A" pin="8"/>
-<wire x1="99.06" y1="17.78" x2="104.14" y2="17.78" width="0.1524" layer="91"/>
-<junction x="104.14" y="20.32"/>
-<wire x1="104.14" y1="20.32" x2="104.14" y2="17.78" width="0.1524" layer="91"/>
-<wire x1="104.14" y1="17.78" x2="106.68" y2="17.78" width="0.1524" layer="91"/>
-<junction x="104.14" y="17.78"/>
-<label x="106.68" y="17.78" size="0.8128" layer="95" xref="yes"/>
 </segment>
 <segment>
@@
 <pinref part="SUPPLY1" gate="GND" pin="GND"/>
 </segment>
+<segment>
+<pinref part="X0" gate="-1" pin="KL"/>
+<wire x1="40.64" y1="223.52" x2="53.34" y2="223.52" width="0.1524" layer="91"/>
+<label x="53.34" y="223.52" size="0.8128" layer="95" xref="yes"/>
+</segment>
+<segment>
+<pinref part="JP1" gate="A" pin="1"/>
+<wire x1="91.44" y1="25.4" x2="86.36" y2="25.4" width="0.1524" layer="91"/>
+<label x="86.36" y="25.4" size="0.8128" layer="95" rot="R180" xref="yes"/>
+</segment>
+<segment>
+<pinref part="JP1" gate="A" pin="3"/>
+<wire x1="91.44" y1="22.86" x2="86.36" y2="22.86" width="0.1524" layer="91"/>
+<label x="86.36" y="22.86" size="0.8128" layer="95" rot="R180" xref="yes"/>
+</segment>
+<segment>
+<pinref part="JP1" gate="A" pin="5"/>
+<wire x1="91.44" y1="20.32" x2="86.36" y2="20.32" width="0.1524" layer="91"/>
+<label x="86.36" y="20.32" size="0.8128" layer="95" rot="R180" xref="yes"/>
+</segment>
+<segment>
+<pinref part="JP1" gate="A" pin="7"/>
+<wire x1="91.44" y1="17.78" x2="86.36" y2="17.78" width="0.1524" layer="91"/>
+<label x="86.36" y="17.78" size="0.8128" layer="95" rot="R180" xref="yes"/>
+</segment>
 </net>
 <net name="VCC" class="2">
@@
 </segment>
 <segment>
-<pinref part="JP1" gate="A" pin="1"/>
-<wire x1="91.44" y1="25.4" x2="86.36" y2="25.4" width="0.1524" layer="91"/>
-<label x="86.36" y="25.4" size="0.8128" layer="95" rot="R180" xref="yes"/>
+<pinref part="JP1" gate="A" pin="2"/>
+<wire x1="99.06" y1="25.4" x2="104.14" y2="25.4" width="0.1524" layer="91"/>
+<label x="104.14" y="25.4" size="0.8128" layer="95" xref="yes"/>
 </segment>
 </net>
@@
 </segment>
 <segment>
-<pinref part="JP1" gate="A" pin="3"/>
-<wire x1="91.44" y1="22.86" x2="86.36" y2="22.86" width="0.1524" layer="91"/>
-<label x="86.36" y="22.86" size="0.8128" layer="95" rot="R180" xref="yes"/>
+<pinref part="JP1" gate="A" pin="4"/>
+<wire x1="99.06" y1="22.86" x2="104.14" y2="22.86" width="0.1524" layer="91"/>
+<label x="104.14" y="22.86" size="0.8128" layer="95" xref="yes"/>
 </segment>
 </net>
@@
 </segment>
 <segment>
-<pinref part="JP1" gate="A" pin="5"/>
-<wire x1="91.44" y1="20.32" x2="86.36" y2="20.32" width="0.1524" layer="91"/>
-<label x="86.36" y="20.32" size="0.8128" layer="95" rot="R180" xref="yes"/>
+<pinref part="JP1" gate="A" pin="6"/>
+<wire x1="99.06" y1="20.32" x2="104.14" y2="20.32" width="0.1524" layer="91"/>
+<label x="104.14" y="20.32" size="0.8128" layer="95" xref="yes"/>
 </segment>
 </net>
@@
 </segment>
 <segment>
-<pinref part="JP1" gate="A" pin="7"/>
-<wire x1="91.44" y1="17.78" x2="86.36" y2="17.78" width="0.1524" layer="91"/>
-<label x="86.36" y="17.78" size="0.8128" layer="95" rot="R180" xref="yes"/>
+<pinref part="JP1" gate="A" pin="8"/>
+<wire x1="99.06" y1="17.78" x2="104.14" y2="17.78" width="0.1524" layer="91"/>
+<label x="104.14" y="17.78" size="0.8128" layer="95" xref="yes"/>
 </segment>
 </net>
@@
 <label x="43.18" y="182.88" size="0.8128" layer="95" rot="R90" xref="yes"/>
 </segment>
-</net>
+<segment>
+<pinref part="X0" gate="-2" pin="KL"/>
+<wire x1="40.64" y1="218.44" x2="53.34" y2="218.44" width="0.1524" layer="91"/>
+<label x="53.34" y="218.44" size="0.8128" layer="95" xref="yes"/>
+</segment>
+</net>

Commit message: Renewal of Port Replicator.
Parts:
- removed J1, J2, J3: AUDIO_JACK_3.5MM_PTH, SparkFun-Connectors:AUDIO_JACK_3.5MM_PTH
- added J21, J22, J23: DIN5, SparkFun-Connectors:DIN5
- added JP6: (no value), pinhead:PINHD-1X3
- added LED4: (no value), led:DUOLED-RG-C
- added S1: (no value), switch-omron:10-XX
- J11, J12, J13: value DIN5 -> AUDIO_JACK_3.5MM_PTH; device SparkFun-Connectors:DIN5 -> SparkFun-Connectors:AUDIO_JACK_3.5MM_PTH
- LED2: value IN -> OUT
- LED3: value OUT -> IN
- renumbered J4 to J14
Connections:
- new net LED0: JP6.1, LED4.AR
- new net LED1: JP6.3, LED4.AG
- net ANLG1R: now also J11.RING; no longer J1.RING
- net ANLG2R: now also J12.RING; no longer J2.RING
- net ANLG3R: now also J13.RING; no longer J3.RING
- net GND: now also J11.SLEEVE, J12.SLEEVE, J13.SLEEVE, J22.2, J23.2, JP6.2, LED4.C, S1.S, S1.S1; no longer J1.SLEEVE, J12.2, J13.2, J2.SLEEVE, J3.SLEEVE
- net MILED: now also LED3.C; no longer LED2.C
- net MIRTN: now also J21.5; no longer J11.5
- net MISND: now also J21.4; no longer J11.4
- net MOLED: now also LED2.C; no longer LED3.C
- net MORTN: now also J23.5; no longer J13.5
- net MOSND: now also J23.4; no longer J13.4
- net MTRTN: now also J22.5; no longer J12.5
- net MTSND: now also J22.4; no longer J12.4
- net RST: now also S1.P, S1.P1
- net VCC/2: now also J11.TIP, J12.TIP, J13.TIP; no longer J1.TIP, J2.TIP, J3.TIP
Other:
- moved on the sheet: LED1, LED2, LED3, R1

Commit message: Silk.
Parts:
- removed LED1: PWR, led:LED3MM
- added LED0/1: (no value), led:DUOLED-RG-C
- LED2: value OUT -> IN
- LED3: value IN -> OUT
- LED4: value (none) -> PWR; device led:DUOLED-RG-C -> led:LED3MM
Connections:
- removed net MILED: LED3.C, R2.2
- removed net MOLED: LED2.C, R3.2
- removed net N$4: LED1.A, R1.1
- new net LEDMI: LED2.C, R2.2
- new net LEDMO: LED3.C, R3.2
- new net LEDPWR: LED4.A, R1.1
- net GND: now also LED0/1.C; no longer LED1.C
- net LED0: now also LED0/1.AR; no longer LED4.AR
- net LED1: now also LED0/1.AG; no longer LED4.AG
Other:
- moved on the sheet: LED2, LED3
Changed lines of the file:
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@@
 <part name="R1" library="rcl" library_urn="urn:adsk.eagle:library:334" deviceset="R-EU_" device="0204/5" package3d_urn="urn:adsk.eagle:package:23488/1"/>
 <part name="R2" library="rcl" library_urn="urn:adsk.eagle:library:334" deviceset="R-EU_" device="0204/5" package3d_urn="urn:adsk.eagle:package:23488/1"/>
-<part name="LED1" library="led" library_urn="urn:adsk.eagle:library:259" deviceset="LED" device="3MM" package3d_urn="urn:adsk.eagle:package:15797/1" value="PWR"/>
-<part name="LED3" library="led" library_urn="urn:adsk.eagle:library:259" deviceset="LED" device="3MM" package3d_urn="urn:adsk.eagle:package:15797/1" value="IN"/>
-<part name="LED2" library="led" library_urn="urn:adsk.eagle:library:259" deviceset="LED" device="3MM" package3d_urn="urn:adsk.eagle:package:15797/1" value="OUT"/>
+<part name="LED4" library="led" library_urn="urn:adsk.eagle:library:259" deviceset="LED" device="3MM" package3d_urn="urn:adsk.eagle:package:15797/1" value="PWR"/>
+<part name="LED2" library="led" library_urn="urn:adsk.eagle:library:259" deviceset="LED" device="3MM" package3d_urn="urn:adsk.eagle:package:15797/1" value="IN"/>
+<part name="LED3" library="led" library_urn="urn:adsk.eagle:library:259" deviceset="LED" device="3MM" package3d_urn="urn:adsk.eagle:package:15797/1" value="OUT"/>
 <part name="R3" library="rcl" library_urn="urn:adsk.eagle:library:334" deviceset="R-EU_" device="0204/5" package3d_urn="urn:adsk.eagle:package:23488/1"/>
 <part name="SUPPLY1" library="supply2" deviceset="GND" device=""/>
@@
 <part name="S1" library="switch-omron" library_urn="urn:adsk.eagle:library:377" deviceset="10-XX" device="" package3d_urn="urn:adsk.eagle:package:27496/1"/>
 <part name="JP6" library="pinhead" library_urn="urn:adsk.eagle:library:325" deviceset="PINHD-1X3" device="" package3d_urn="urn:adsk.eagle:package:22458/2"/>
-<part name="LED4" library="led" library_urn="urn:adsk.eagle:library:259" deviceset="DUOLED-RG-C" device="" package3d_urn="urn:adsk.eagle:package:15851/1"/>
+<part name="LED0/1" library="led" library_urn="urn:adsk.eagle:library:259" deviceset="DUOLED-RG-C" device="" package3d_urn="urn:adsk.eagle:package:15851/1"/>
 </parts>
 <sheets>
@@
 <attribute name="VALUE" x="255.27" y="154.178" size="1.778" layer="96"/>
 </instance>
-<instance part="LED1" gate="G$1" x="35.56" y="167.64" smashed="yes">
+<instance part="LED4" gate="G$1" x="35.56" y="167.64" smashed="yes">
 <attribute name="NAME" x="39.116" y="163.068" size="1.778" layer="95" rot="R90"/>
 <attribute name="VALUE" x="41.275" y="163.068" size="1.778" layer="96" rot="R90"/>
 </instance>
-<instance part="LED3" gate="G$1" x="271.78" y="157.48" smashed="yes" rot="R270">
+<instance part="LED2" gate="G$1" x="271.78" y="157.48" smashed="yes" rot="R270">
 <attribute name="NAME" x="267.208" y="153.924" size="1.778" layer="95"/>
 <attribute name="VALUE" x="267.208" y="151.765" size="1.778" layer="96"/>
 </instance>
-<instance part="LED2" gate="G$1" x="271.78" y="139.7" smashed="yes" rot="R270">
+<instance part="LED3" gate="G$1" x="271.78" y="139.7" smashed="yes" rot="R270">
 <attribute name="NAME" x="267.208" y="136.144" size="1.778" layer="95"/>
 <attribute name="VALUE" x="267.208" y="133.985" size="1.778" layer="96"/>
@@
 <attribute name="VALUE" x="39.37" y="45.72" size="1.778" layer="96" rot="MR0"/>
 </instance>
-<instance part="LED4" gate="G$1" x="58.42" y="170.18" smashed="yes">
+<instance part="LED0/1" gate="G$1" x="58.42" y="170.18" smashed="yes">
 <attribute name="NAME" x="64.77" y="165.1" size="1.778" layer="95" rot="R90"/>
 <attribute name="VALUE" x="67.31" y="165.1" size="1.778" layer="96" rot="R90"/>
@@
 </segment>
 <segment>
-<pinref part="LED1" gate="G$1" pin="C"/>
+<pinref part="LED4" gate="G$1" pin="C"/>
 <wire x1="35.56" y1="162.56" x2="35.56" y2="160.02" width="0.1524" layer="91"/>
 <label x="35.56" y="160.02" size="0.8128" layer="95" rot="R270" xref="yes"/>
@@
 </segment>
 <segment>
-<pinref part="LED4" gate="G$1" pin="C"/>
+<pinref part="LED0/1" gate="G$1" pin="C"/>
 <wire x1="55.88" y1="170.18" x2="53.34" y2="170.18" width="0.1524" layer="91"/>
 <label x="53.34" y="170.18" size="0.8128" layer="95" rot="R180" xref="yes"/>
@@
 </segment>
 <segment>
+<pinref part="LED2" gate="G$1" pin="A"/>
+<wire x1="279.4" y1="157.48" x2="276.86" y2="157.48" width="0.1524" layer="91"/>
 <pinref part="LED3" gate="G$1" pin="A"/>
-<wire x1="279.4" y1="157.48" x2="276.86" y2="157.48" width="0.1524" layer="91"/>
-<pinref part="LED2" gate="G$1" pin="A"/>
 <wire x1="276.86" y1="157.48" x2="274.32" y2="157.48" width="0.1524" layer="91"/>
 <wire x1="274.32" y1="139.7" x2="276.86" y2="139.7" width="0.1524" layer="91"/>
@@
 </segment>
 </net>
-<net name="MILED" class="0">
-<segment>
-<pinref part="LED3" gate="G$1" pin="C"/>
+<net name="LEDMI" class="0">
+<segment>
+<pinref part="LED2" gate="G$1" pin="C"/>
 <pinref part="R2" gate="G$1" pin="2"/>
 <wire x1="266.7" y1="157.48" x2="264.16" y2="157.48" width="0.1524" layer="91"/>
 </segment>
 </net>
-<net name="MOLED" class="0">
-<segment>
-<pinref part="LED2" gate="G$1" pin="C"/>
+<net name="LEDMO" class="0">
+<segment>
+<pinref part="LED3" gate="G$1" pin="C"/>
 <pinref part="R3" gate="G$1" pin="2"/>
 <wire x1="266.7" y1="139.7" x2="264.16" y2="139.7" width="0.1524" layer="91"/>
 </segment>
 </net>
-<net name="N$4" class="0">
+<net name="LEDPWR" class="0">
 <segment>
 <pinref part="R1" gate="G$1" pin="1"/>
-<pinref part="LED1" gate="G$1" pin="A"/>
+<pinref part="LED4" gate="G$1" pin="A"/>
 <wire x1="35.56" y1="172.72" x2="35.56" y2="170.18" width="0.1524" layer="91"/>
 </segment>
@@
 <net name="LED0" class="0">
 <segment>
-<pinref part="LED4" gate="G$1" pin="AR"/>
+<pinref part="LED0/1" gate="G$1" pin="AR"/>
 <wire x1="58.42" y1="177.8" x2="58.42" y2="180.34" width="0.1524" layer="91"/>
 <label x="58.42" y="180.34" size="0.8128" layer="95" rot="R90" xref="yes"/>
@@
 <net name="LED1" class="0">
 <segment>
-<pinref part="LED4" gate="G$1" pin="AG"/>
+<pinref part="LED0/1" gate="G$1" pin="AG"/>
 <wire x1="58.42" y1="162.56" x2="58.42" y2="160.02" width="0.1524" layer="91"/>
 <label x="58.42" y="160.02" size="0.8128" layer="95" rot="R270" xref="yes"/>
