File: peripheral/port-replicator/hardware/logicboard/p20-001.sch (EAGLE design)
At the start: 25 parts, among them IC1 74ALS04N, J0 DC9V, J11 AUDIO_JACK_3.5MM_PTH, J12 AUDIO_JACK_3.5MM_PTH, J13 AUDIO_JACK_3.5MM_PTH, J14 AUDIO_JACK_3.5MM_PTH, J7 DIN5, J8 DIN5, J9 DIN5, X0 MKDSN1,5/2-5,08

Commit message: Redesign of port rep.
Parts:
- removed JP1: (no value), adafruit:PINHD-2X4
- added RN1, RN2: (no value), resistor-net:RN04
- added S2: (no value), switch-dil:DIP04S
Connections:
- new net N$5: RN2.2, S2-1.2
- new net N$6: RN2.3, S2-2.2
- new net N$7: RN2.4, S2-3.2
- new net N$8: RN2.5, S2-4.2
- net DTCT1: now also J11.TSH, RN1.2, S2-1.1; no longer JP1.2
- net DTCT2: now also J12.TSH, RN1.3, S2-2.1; no longer JP1.4
- net DTCT3: now also J13.TSH, RN1.4, S2-3.1; no longer JP1.6
- net DTCT4: now also J14.TSH, RN1.5, S2-4.1; no longer JP1.8
- net GND: now also RN1.1; no longer JP1.1, JP1.3, JP1.5, JP1.7
- net VCC/2: now also RN2.1
Changed lines of the file:
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@@
 <part name="J13" library="SparkFun-Connectors" library_urn="urn:adsk.eagle:library:513" deviceset="AUDIO_JACK_3.5MM" device="_PTH" package3d_urn="urn:adsk.eagle:package:37997/1"/>
 <part name="J14" library="SparkFun-Connectors" library_urn="urn:adsk.eagle:library:513" deviceset="AUDIO_JACK_3.5MM" device="_PTH" package3d_urn="urn:adsk.eagle:package:37997/1"/>
-<part name="JP1" library="adafruit" library_urn="urn:adsk.eagle:library:420" deviceset="PINHD-2X4" device="" package3d_urn="urn:adsk.eagle:package:6240893/1"/>
 <part name="IC1" library="74xx-us" library_urn="urn:adsk.eagle:library:88" deviceset="74*04" device="N" package3d_urn="urn:adsk.eagle:package:16407/2" technology="ALS" value="74ALS04N"/>
 <part name="R1" library="rcl" library_urn="urn:adsk.eagle:library:334" deviceset="R-EU_" device="0204/5" package3d_urn="urn:adsk.eagle:package:23488/1"/>
@@
 <part name="JP6" library="pinhead" library_urn="urn:adsk.eagle:library:325" deviceset="PINHD-1X3" device="" package3d_urn="urn:adsk.eagle:package:22458/2"/>
 <part name="LED0/1" library="led" library_urn="urn:adsk.eagle:library:259" deviceset="DUOLED-RG-C" device="" package3d_urn="urn:adsk.eagle:package:15851/1"/>
+<part name="RN1" library="resistor-net" library_urn="urn:adsk.eagle:library:343" deviceset="RN04" device="" package3d_urn="urn:adsk.eagle:package:24976/1"/>
+<part name="SUPPLY2" library="supply2" deviceset="GND" device=""/>
+<part name="S2" library="switch-dil" library_urn="urn:adsk.eagle:library:375" deviceset="DIP04S" device="" package3d_urn="urn:adsk.eagle:package:27250/2"/>
+<part name="RN2" library="resistor-net" library_urn="urn:adsk.eagle:library:343" deviceset="RN04" device="" package3d_urn="urn:adsk.eagle:package:24976/1"/>
 </parts>
 <sheets>
@@
 <attribute name="VALUE" x="86.36" y="45.72" size="1.778" layer="96" font="vector"/>
 </instance>
-<instance part="JP1" gate="A" x="93.98" y="20.32" smashed="yes">
-<attribute name="NAME" x="87.63" y="28.575" size="1.778" layer="95"/>
-<attribute name="VALUE" x="87.63" y="12.7" size="1.778" layer="96"/>
-</instance>
 <instance part="IC1" gate="A" x="210.82" y="157.48" smashed="yes">
 <attribute name="NAME" x="213.36" y="160.655" size="1.778" layer="95"/>
@@
 <attribute name="NAME" x="64.77" y="165.1" size="1.778" layer="95" rot="R90"/>
 <attribute name="VALUE" x="67.31" y="165.1" size="1.778" layer="96" rot="R90"/>
+</instance>
+<instance part="RN1" gate="1" x="83.82" y="17.78" smashed="yes" rot="R90">
+<attribute name="NAME" x="81.28" y="15.24" size="1.778" layer="95" rot="R90"/>
+<attribute name="VALUE" x="88.138" y="15.24" size="1.778" layer="96" rot="R90"/>
+</instance>
+<instance part="SUPPLY2" gate="GND" x="83.82" y="7.62" smashed="yes"/>
+<instance part="S2" gate="-1" x="162.56" y="71.12" smashed="yes">
+<attribute name="NAME" x="165.1" y="67.31" size="1.778" layer="95" rot="R90"/>
+</instance>
+<instance part="S2" gate="-2" x="167.64" y="71.12" smashed="yes">
+<attribute name="NAME" x="170.18" y="67.31" size="1.778" layer="95" rot="R90"/>
+</instance>
+<instance part="S2" gate="-3" x="172.72" y="71.12" smashed="yes">
+<attribute name="NAME" x="175.26" y="67.31" size="1.778" layer="95" rot="R90"/>
+</instance>
+<instance part="S2" gate="-4" x="177.8" y="71.12" smashed="yes">
+<attribute name="NAME" x="180.34" y="67.31" size="1.778" layer="95" rot="R90"/>
+<attribute name="VALUE" x="182.88" y="67.31" size="1.778" layer="96" rot="R90"/>
+</instance>
+<instance part="RN2" gate="1" x="157.48" y="83.82" smashed="yes">
+<attribute name="NAME" x="154.94" y="86.36" size="1.778" layer="95"/>
+<attribute name="VALUE" x="154.94" y="79.502" size="1.778" layer="96"/>
 </instance>
 </instances>
@@
 </segment>
 <segment>
-<pinref part="JP1" gate="A" pin="1"/>
-<wire x1="91.44" y1="25.4" x2="86.36" y2="25.4" width="0.1524" layer="91"/>
-<label x="86.36" y="25.4" size="0.8128" layer="95" rot="R180" xref="yes"/>
-</segment>
-<segment>
-<pinref part="JP1" gate="A" pin="3"/>
-<wire x1="91.44" y1="22.86" x2="86.36" y2="22.86" width="0.1524" layer="91"/>
-<label x="86.36" y="22.86" size="0.8128" layer="95" rot="R180" xref="yes"/>
-</segment>
-<segment>
-<pinref part="JP1" gate="A" pin="5"/>
-<wire x1="91.44" y1="20.32" x2="86.36" y2="20.32" width="0.1524" layer="91"/>
-<label x="86.36" y="20.32" size="0.8128" layer="95" rot="R180" xref="yes"/>
-</segment>
-<segment>
-<pinref part="JP1" gate="A" pin="7"/>
-<wire x1="91.44" y1="17.78" x2="86.36" y2="17.78" width="0.1524" layer="91"/>
-<label x="86.36" y="17.78" size="0.8128" layer="95" rot="R180" xref="yes"/>
-</segment>
-<segment>
 <pinref part="S1" gate="1" pin="S"/>
 <wire x1="162.56" y1="200.66" x2="165.1" y2="200.66" width="0.1524" layer="91"/>
@@
 <label x="309.88" y="104.14" size="0.8128" layer="95" rot="MR0" xref="yes"/>
 </segment>
+<segment>
+<pinref part="RN1" gate="1" pin="1"/>
+<wire x1="83.82" y1="12.7" x2="83.82" y2="10.16" width="0.1524" layer="91"/>
+<pinref part="SUPPLY2" gate="GND" pin="GND"/>
+</segment>
 </net>
 <net name="VCC" class="2">
@@
 </segment>
 <segment>
-<pinref part="JP1" gate="A" pin="2"/>
-<wire x1="99.06" y1="25.4" x2="104.14" y2="25.4" width="0.1524" layer="91"/>
-<label x="104.14" y="25.4" size="0.8128" layer="95" xref="yes"/>
+<pinref part="J11" gate="G$1" pin="TSH"/>
+<wire x1="96.52" y1="132.08" x2="99.06" y2="132.08" width="0.1524" layer="91"/>
+<label x="99.06" y="132.08" size="0.8128" layer="95" xref="yes"/>
+</segment>
+<segment>
+<pinref part="RN1" gate="1" pin="2"/>
+<wire x1="83.82" y1="22.86" x2="86.36" y2="22.86" width="0.1524" layer="91"/>
+<label x="86.36" y="22.86" size="0.8128" layer="95" xref="yes"/>
+</segment>
+<segment>
+<pinref part="S2" gate="-1" pin="1"/>
+<wire x1="162.56" y1="66.04" x2="162.56" y2="60.96" width="0.1524" layer="91"/>
+<label x="162.56" y="60.96" size="0.8128" layer="95" rot="R270" xref="yes"/>
 </segment>
 </net>
@@
 </segment>
 <segment>
-<pinref part="JP1" gate="A" pin="4"/>
-<wire x1="99.06" y1="22.86" x2="104.14" y2="22.86" width="0.1524" layer="91"/>
-<label x="104.14" y="22.86" size="0.8128" layer="95" xref="yes"/>
+<pinref part="J12" gate="G$1" pin="TSH"/>
+<wire x1="96.52" y1="104.14" x2="99.06" y2="104.14" width="0.1524" layer="91"/>
+<label x="99.06" y="104.14" size="0.8128" layer="95" xref="yes"/>
+</segment>
+<segment>
+<pinref part="RN1" gate="1" pin="3"/>
+<wire x1="83.82" y1="27.94" x2="86.36" y2="27.94" width="0.1524" layer="91"/>
+<label x="86.36" y="27.94" size="0.8128" layer="95" xref="yes"/>
+</segment>
+<segment>
+<pinref part="S2" gate="-2" pin="1"/>
+<wire x1="167.64" y1="66.04" x2="167.64" y2="60.96" width="0.1524" layer="91"/>
+<label x="167.64" y="60.96" size="0.8128" layer="95" rot="R270" xref="yes"/>
 </segment>
 </net>
@@
 </segment>
 <segment>
-<pinref part="JP1" gate="A" pin="6"/>
-<wire x1="99.06" y1="20.32" x2="104.14" y2="20.32" width="0.1524" layer="91"/>
-<label x="104.14" y="20.32" size="0.8128" layer="95" xref="yes"/>
+<pinref part="J13" gate="G$1" pin="TSH"/>
+<wire x1="96.52" y1="81.28" x2="99.06" y2="81.28" width="0.1524" layer="91"/>
+<label x="99.06" y="81.28" size="0.8128" layer="95" xref="yes"/>
+</segment>
+<segment>
+<pinref part="RN1" gate="1" pin="4"/>
+<wire x1="83.82" y1="33.02" x2="86.36" y2="33.02" width="0.1524" layer="91"/>
+<label x="86.36" y="33.02" size="0.8128" layer="95" xref="yes"/>
+</segment>
+<segment>
+<pinref part="S2" gate="-3" pin="1"/>
+<wire x1="172.72" y1="66.04" x2="172.72" y2="60.96" width="0.1524" layer="91"/>
+<label x="172.72" y="60.96" size="0.8128" layer="95" rot="R270" xref="yes"/>
 </segment>
 </net>
@@
 </segment>
 <segment>
-<pinref part="JP1" gate="A" pin="8"/>
-<wire x1="99.06" y1="17.78" x2="104.14" y2="17.78" width="0.1524" layer="91"/>
-<label x="104.14" y="17.78" size="0.8128" layer="95" xref="yes"/>
+<pinref part="J14" gate="G$1" pin="TSH"/>
+<wire x1="96.52" y1="50.8" x2="99.06" y2="50.8" width="0.1524" layer="91"/>
+<label x="99.06" y="50.8" size="0.8128" layer="95" xref="yes"/>
+</segment>
+<segment>
+<pinref part="RN1" gate="1" pin="5"/>
+<wire x1="83.82" y1="38.1" x2="86.36" y2="38.1" width="0.1524" layer="91"/>
+<label x="86.36" y="38.1" size="0.8128" layer="95" xref="yes"/>
+</segment>
+<segment>
+<pinref part="S2" gate="-4" pin="1"/>
+<wire x1="177.8" y1="66.04" x2="177.8" y2="60.96" width="0.1524" layer="91"/>
+<label x="177.8" y="60.96" size="0.8128" layer="95" rot="R270" xref="yes"/>
 </segment>
 </net>
@@
 <label x="99.06" y="48.26" size="0.8128" layer="95" xref="yes"/>
 </segment>
+<segment>
+<pinref part="RN2" gate="1" pin="1"/>
+<wire x1="152.4" y1="83.82" x2="149.86" y2="83.82" width="0.1524" layer="91"/>
+<label x="149.86" y="83.82" size="0.8128" layer="95" rot="R180" xref="yes"/>
+</segment>
 </net>
 <net name="MISND" class="0">
@@
 </segment>
 </net>
+<net name="N$5" class="0">
+<segment>
+<pinref part="RN2" gate="1" pin="2"/>
+<pinref part="S2" gate="-1" pin="2"/>
+<wire x1="162.56" y1="83.82" x2="162.56" y2="76.2" width="0.1524" layer="91"/>
+</segment>
+</net>
+<net name="N$6" class="0">
+<segment>
+<pinref part="RN2" gate="1" pin="3"/>
+<pinref part="S2" gate="-2" pin="2"/>
+<wire x1="167.64" y1="83.82" x2="167.64" y2="76.2" width="0.1524" layer="91"/>
+</segment>
+</net>
+<net name="N$7" class="0">
+<segment>
+<pinref part="RN2" gate="1" pin="4"/>
+<pinref part="S2" gate="-3" pin="2"/>
+<wire x1="172.72" y1="83.82" x2="172.72" y2="76.2" width="0.1524" layer="91"/>
+</segment>
+</net>
+<net name="N$8" class="0">
+<segment>
+<pinref part="RN2" gate="1" pin="5"/>
+<pinref part="S2" gate="-4" pin="2"/>
+<wire x1="177.8" y1="83.82" x2="177.8" y2="76.2" width="0.1524" layer="91"/>
+</segment>
+</net>
